Commit message: Fix jawbot Gazebo URDF/SDF wheel alignment, caster clearance, and joint state TF bridge

File: jawbot_description/urdf/jawbot.urdf.xacro (robot description, xacro)
@@ -81,8 +81,8 @@
   </link>
   <joint name="left_wheel_joint" type="continuous">
-    <origin xyz="-0.00079275 0.0925 -0.060292" rpy="0 0 0" />
+    <origin xyz="-0.00079275 0.0925 -0.061542" rpy="0 0 0" />
     <parent link="base_link" />
     <child link="left_wheel_link" />
-    <axis xyz="0 -1 0" />
+    <axis xyz="0 1 0" />
   </joint>
   <!-- ============================================================================= -->
@@ -112,5 +112,5 @@
   </link>
   <joint name="right_wheel_joint" type="continuous">
-    <origin xyz="-0.00079275 -0.095321 -0.060292" rpy="0 0 0" />
+    <origin xyz="-0.00079275 -0.095321 -0.061542" rpy="0 0 0" />
     <parent link="base_link" />
     <child link="right_wheel_link" />
