Commit message: feat: integrate GY-87 IMU into firmware and ROS 2 hardware interface

File: jawbot_description/urdf/jawbot.urdf.xacro (robot description, xacro)
@@ -270,3 +270,22 @@
     <axis xyz="0 0 0" />
   </joint>
+  <!-- ============================================================================= -->
+  <!-- IMU SENSOR                                                                    -->
+  <!-- ============================================================================= -->
+<link name="imu_link">
+  <visual>
+    <geometry>
+      <box size="0.02 0.02 0.01"/> <!-- Small box representing the GY-87 -->
+    </geometry>
+    <material name="red">
+      <color rgba="1.0 0.0 0.0 1.0"/>
+    </material>
+  </visual>
+</link>
+<!-- IMU Joint: Middle of robot, 6cm (0.06m) high -->
+<joint name="imu_joint" type="fixed">
+  <parent link="base_link"/> <!-- Assuming your main chassis is base_link -->
+  <child link="imu_link"/>
+  <origin xyz="0 0 0.06" rpy="0 0 0"/>
+</joint>
 </robot>

File: jawbot_description/urdf/jawbot_ros2_control.urdf.xacro (robot description, xacro)
@@ -19,4 +19,12 @@
       <state_interface name="velocity"/>
     </joint>
+    <sensor name="imu_sensor">
+    <state_interface name="linear_acceleration.x"/>
+    <state_interface name="linear_acceleration.y"/>
+    <state_interface name="linear_acceleration.z"/>
+    <state_interface name="angular_velocity.x"/>
+    <state_interface name="angular_velocity.y"/>
+    <state_interface name="angular_velocity.z"/>
+    </sensor>
   </ros2_control>
 </robot>
